Commit message: Finish first draft of  gordon_description

File: src/gordon_description/urdf/gordon_description.urdf (robot description, URDF)
Before this commit: robot gordon, 2 links, 1 joints
Links:
- added link camera_link; visual box size=${camera_length} ${camera_width} ${camera_height}
- added link caster_link; visual sphere radius=${caster_radius}
- added link gate_link; visual box size=${gate_length} ${gate_width} ${gate_height}
Joints:
- added joint camera_joint: type fixed, parent base_link, child camera_link, origin xyz=${camera_x_offset} 0 ${camera_z_offset} rpy=0 ${camera_pitch} 0
- added joint caster_joint: type fixed, parent base_link, child caster_link, origin xyz=${caster_x_offset} 0 ${-caster_z_offset} rpy=0 0 0
- added joint gate_joint: type continuous, parent base_link, child gate_link, origin xyz=${gate_x_offset} 0 ${gate_z_offset} rpy=0 0 0, axis 0 1 0
- joint base_joint: origin xyz=0.0 0.0 0.0 rpy=0 0 0 -> xyz=0 0 ${-footprint_z_offset} rpy=0 0 0
