Commit message: Create launch files for test purposes

File: src/gordon_description/urdf/robot.urdf (robot description, URDF)
Before this commit: robot gordon, 5 links, 4 joints
Joints:
- joint camera_joint: origin xyz=${camera_x_offset} 0 ${camera_z_offset} rpy=0 ${camera_pitch} 0 -> xyz=${camera_x_offset} 0 ${camera_z_offset} rpy=${camera_roll} ${camera_pitch} ${camera_yaw}

Commit message: Add test images and minor changes

File: src/gordon_description/urdf/robot.urdf (robot description, URDF)
Before this commit: robot gordon, 5 links, 4 joints
Joints:
- joint camera_joint: origin xyz=${camera_x_offset} 0 ${camera_z_offset} rpy=${camera_roll} ${camera_pitch} ${camera_yaw} -> xyz=${camera_x_offset} 0 ${camera_z_offset} rpy=${camera_roll} 0 ${camera_yaw}
