Commit message: 4

File: src/gordon_description/urdf/gordon.urdf (robot description, URDF)
Before this commit: robot gordon, 7 links, 6 joints
Joints:
- joint sonar_front_joint: origin xyz=${front_sensor_x_offset} {front_sensor_y_offset} {front_sensor_z_offset} rpy=0 0 0 -> xyz=${front_sensor_x_offset} ${front_sensor_y_offset} ${front_sensor_z_offset} rpy=0 0 0
- joint sonar_left_joint: origin xyz=${left_sensor_x_offset} {left_sensor_y_offset} {left_sensor_z_offset} rpy=0 0 0 -> xyz=${left_sensor_x_offset} ${left_sensor_y_offset} ${left_sensor_z_offset} rpy=0 0 0

Commit message: 9

File: src/gordon_description/urdf/gordon.urdf (robot description, URDF)
Before this commit: robot gordon, 7 links, 6 joints
Joints:
- joint sonar_left_joint: origin xyz=${left_sensor_x_offset} ${left_sensor_y_offset} ${left_sensor_z_offset} rpy=0 0 0 -> xyz=${left_sensor_x_offset} ${left_sensor_y_offset} ${left_sensor_z_offset} rpy=0 0 1.5707
